File: KiCad/ElectronicLoad.kicad_pcb (KiCad board)
At the start: 2 copper layers, 99.8 x 99.8 mm, 164 parts, among them J1 LOAD, J4 12V, J5 USB, J6 PROG, M1 FAN, Q1 any, Q2 any, Q3 BSS138, Q4 PMOS, Q5 BSS138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

Commit message: rev0.2: adjust component values
Parts:
- C1, C2: value 1nF (tbd) -> 4.7nF
- C11, C12: value 22pF (tbd) -> 100pF
- C13, C14: value 22pF (tbd) -> 4.7nF
- C19: value 3.3pF (tbd) -> 100pF
- C21: value 100pF (tbd) -> 4.7nF
- D2: value D_Small -> Schottky
- R12, R13, R14, R15, R16, R17, R18, R19, R20, R201, R21, R22, R23, R24, R38: value R_Small -> 2k (1%)
- R25, R26, R27, R28, R29, R30, R31, R32, R33, R34, R35, R36, R37: value R_Small -> 1k (1%)
- R40, R42, R44, R49: value 1M -> 100k
- R41: value 0* -> 0
- R46: value 470k* -> 100k (1%)
- R47: value 10k* -> 10k (1%)
- R65, R69: value 1ohm -> 10
- R66: value 2.2k -> 3.3k
- R67: value 3.3k -> 10k
- R68: value 12k -> 22k
- R70: value R_Small -> 0
- R88, R89: value 1 -> 10
- R93: value 10 -> dnp
- R95: value 1ohm -> dnp
- R96: value dnp -> 1ohm
Changed lines of the file:
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@@
 			)
 		)
-		(property "Value" "1M"
+		(property "Value" "100k"
 			(at 0 1.43 0)
 			(layer "F.Fab")
@@
 		(tags "resistor")
 		(property "Reference" "R64"
-			(at 2.9 -0.84 90)
+			(at 2.51 0.02 180)
 			(layer "F.SilkS")
 			(effects
@@
 			)
 		)
-		(property "Value" "1M"
+		(property "Value" "100k"
 			(at 0 1.43 0)
 			(layer "F.Fab")
@@
 			)
 		)
-		(property "Value" "22pF (tbd)"
+		(property "Value" "4.7nF"
 			(at 0 -1.43 90)
 			(layer "B.Fab")
@@
 			)
 		)
-		(property "Value" "R_Small"
+		(property "Value" "2k (1%)"
 			(at 0 -1.43 90)
 			(layer "B.Fab")
@@
 			)
 		)
-		(property "Value" "R_Small"
+		(property "Value" "1k (1%)"
 			(at 0 -1.43 90)
 			(layer "B.Fab")
@@
 			)
 		)
-		(property "Value" "10k*"
+		(property "Value" "10k (1%)"
 			(at 0 -1.43 0)
 			(layer "B.Fab")
@@
 			)
 		)
-		(property "Value" "1ohm"
+		(property "Value" "10"
 			(at 0 -1.43 0)
 			(layer "B.Fab")
@@
 			)
 		)
-		(property "Value" "3.3pF (tbd)"
+		(property "Value" "100pF"
 			(at 0 -1.43 90)
 			(layer "B.Fab")
@@
 			)
 		)
-		(property "Value" "R_Small"
+		(property "Value" "0"
 			(at 0 -1.43 90)
 			(layer "B.Fab")
@@
 			)
 		)
-		(property "Value" "R_Small"
+		(property "Value" "1k (1%)"
 			(at 0 -1.43 90)
 			(layer "B.Fab")
@@
 			)
 		)
-		(property "Value" "R_Small"
+		(property "Value" "1k (1%)"
 			(at 0 -1.43 90)
 			(layer "B.Fab")
@@
 			)
 		)
-		(property "Value" "R_Small"
+		(property "Value" "2k (1%)"
 			(at 0 -1.43 90)
 			(layer "B.Fab")
@@
 			)
 		)
-		(property "Value" "R_Small"
+		(property "Value" "1k (1%)"
 			(at 0 -1.43 90)
 			(layer "B.Fab")
@@
 			)
 		)
-		(property "Value" "3.3k"
+		(property "Value" "10k"
 			(at 0 -1.65 90)
 			(layer "B.Fab")
@@
 			)
 		)
-		(property "Value" "R_Small"
+		(property "Value" "2k (1%)"
 			(at 0 -1.43 90)
 			(layer "B.Fab")
@@
 			)
 		)
-		(property "Value" "470k*"
+		(property "Value" "100k (1%)"
 			(at 0 -1.43 0)
 			(layer "B.Fab")
@@
 			)
 		)
-		(property "Value" "R_Small"
+		(property "Value" "2k (1%)"
 			(at 0 -1.43 90)
 			(layer "B.Fab")
@@
 			)
 		)
-		(property "Value" "12k"
+		(property "Value" "22k"
 			(at 0 -1.65 90)
 			(layer "B.Fab")
@@
 			)
 		)
-		(property "Value" "R_Small"
+		(property "Value" "2k (1%)"
 			(at 0 -1.43 90)
 			(layer "B.Fab")
@@
 			)
 		)
-		(property "Value" "R_Small"
+		(property "Value" "1k (1%)"
 			(at 0 -1.43 90)
 			(layer "B.Fab")
@@
 			)
 		)
-		(property "Value" "R_Small"
+		(property "Value" "1k (1%)"
 			(at 0 -1.43 90)
 			(layer "B.Fab")
@@
 			)
 		)
-		(property "Value" "22pF (tbd)"
+		(property "Value" "100pF"
 			(at 0 -1.43 90)
 			(layer "B.Fab")
@@
 			)
 		)
-		(property "Value" "R_Small"
+		(property "Value" "2k (1%)"
 			(at 0 -1.43 90)
 			(layer "B.Fab")
@@
 			)
 		)
-		(property "Value" "1nF (tbd)"
+		(property "Value" "4.7nF"
 			(at 0 -1.43 180)
 			(layer "B.Fab")
@@
 			)
 		)
-		(property "Value" "2.2k"
+		(property "Value" "3.3k"
 			(at 0 -1.65 90)
 			(layer "B.Fab")
@@
 			)
 		)
-		(property "Value" "R_Small"
+		(property "Value" "2k (1%)"
 			(at 0 -1.43 90)
 			(layer "B.Fab")
@@
 			)
 		)
-		(property "Value" "R_Small"
+		(property "Value" "2k (1%)"
 			(at 0 -1.43 90)
 			(layer "B.Fab")
@@
 			)
 		)
-		(property "Value" "R_Small"
+		(property "Value" "1k (1%)"
 			(at 0 -1.43 90)
 			(layer "B.Fab")
@@
 			)
 		)
-		(property "Value" "22pF (tbd)"
+		(property "Value" "100pF"
 			(at 0 -1.43 90)
 			(layer "B.Fab")
@@
 			)
 		)
-		(property "Value" "1ohm"
+		(property "Value" "dnp"
 			(at 0 -1.65 90)
 			(layer "B.Fab")
@@
 			)
 		)
-		(property "Value" "1M"
+		(property "Value" "100k"
 			(at 0 -1.43 90)
 			(layer "B.Fab")
@@
 			)
 		)
-		(property "Value" "100pF (tbd)"
+		(property "Value" "4.7nF"
 			(at 0 -1.43 0)
 			(layer "B.Fab")
@@
 			)
 		)
-		(property "Value" "1ohm"
+		(property "Value" "10"
 			(at 0 -1.43 90)
 			(layer "B.Fab")
@@
 			)
 		)
-		(property "Value" "R_Small"
+		(property "Value" "2k (1%)"
 			(at 0 -1.43 90)
 			(layer "B.Fab")
@@
 			)
 		)
-		(property "Value" "1M"
+		(property "Value" "100k"
 			(at 0 -1.43 90)
 			(layer "B.Fab")
@@
 			)
 		)
-		(property "Value" "R_Small"
+		(property "Value" "2k (1%)"
 			(at 0 -1.43 90)
 			(layer "B.Fab")
@@
 			)
 		)
-		(property "Value" "10"
+		(property "Value" "dnp"
 			(at 0 -1.65 90)
 			(layer "B.Fab")
@@
 			)
 		)
-		(property "Value" "R_Small"
+		(property "Value" "1k (1%)"
 			(at 0 -1.43 90)
 			(layer "B.Fab")
@@
 			)
 		)
-		(property "Value" "0*"
+		(property "Value" "0"
 			(at 0 -1.43 0)
 			(layer "B.Fab")
@@
 			)
 		)
-		(property "Value" "R_Small"
+		(property "Value" "2k (1%)"
 			(at 0 -1.43 90)
 			(layer "B.Fab")
@@
 			)
 		)
-		(property "Value" "R_Small"
+		(property "Value" "1k (1%)"
 			(at 0 -1.43 90)
 			(layer "B.Fab")
@@
 			)
 		)
-		(property "Value" "R_Small"
+		(property "Value" "1k (1%)"
 			(at 0 -1.43 90)
 			(layer "B.Fab")
@@
 			)
 		)
-		(property "Value" "R_Small"
+		(property "Value" "2k (1%)"
 			(at 0 -1.43 90)
 			(layer "B.Fab")
@@
 			)
 		)
-		(property "Value" "D_Small"
+		(property "Value" "Schottky"
 			(at 0 -2.1 0)
 			(layer "B.Fab")
@@
 			)
 		)
-		(property "Value" "dnp"
+		(property "Value" "1ohm"
 			(at 0 -1.65 90)
 			(layer "B.Fab")
@@
 			)
 		)
-		(property "Value" "1"
+		(property "Value" "10"
 			(at 0 -1.43 90)
 			(layer "B.Fab")
@@
 			)
 		)
-		(property "Value" "R_Small"
+		(property "Value" "2k (1%)"
 			(at 0 -1.43 90)
 			(layer "B.Fab")
@@
 			)
 		)
-		(property "Value" "R_Small"
+		(property "Value" "1k (1%)"
 			(at 0 -1.43 90)
 			(layer "B.Fab")
@@
 			)
 		)
-		(property "Value" "1nF (tbd)"
+		(property "Value" "4.7nF"
 			(at 0 -1.43 180)
 			(layer "B.Fab")
@@
 			)
 		)
-		(property "Value" "1"
+		(property "Value" "10"
 			(at 0 -1.43 90)
 			(layer "B.Fab")
@@
 			)
 		)
-		(property "Value" "R_Small"
+		(property "Value" "2k (1%)"
 			(at 0 -1.43 90)
 			(layer "B.Fab")
@@
 			)
 		)
-		(property "Value" "R_Small"
+		(property "Value" "2k (1%)"
 			(at 0 -1.43 90)
 			(layer "B.Fab")
@@
 			)
 		)
-		(property "Value" "22pF (tbd)"
+		(property "Value" "4.7nF"
 			(at 0 -1.43 90)
 			(layer "B.Fab")
@@
 			)
 		)
-		(property "Value" "R_Small"
+		(property "Value" "1k (1%)"
 			(at 0 -1.43 90)
 			(layer "B.Fab")
@@
 			)
 		)
-		(property "Value" "R_Small"
+		(property "Value" "1k (1%)"
 			(at 0 -1.43 90)
 			(layer "B.Fab")

Commit message: rev 0.2 schematics + pcb adjustments
Parts:
- R41: value 0 -> 100k (1%)
- R46: value 100k (1%) -> 20k (1%)
- R47: value 10k (1%) -> 4.7k (1%)
- R52, R53: value 22 -> dnp
- R74: value 20k -> 0
- R75: value 10k -> dnp
- R81: value 0 -> 10
- R83, R84: value 10k -> 470
- RS1, RS2: value 0.001 -> 0.010
Connections:
- U5 pad 12: unconnected-(U5-GPIO8/TOUCH8/ADC1_CH7-Pad12) -> PWR_C_SET_EN
- U5 pad 16: PWR_C_SET_EN -> unconnected-(U5-GPIO46-Pad16)
Routing:
- net PWR_C_SET_EN: track 72.5 -> 77.5 mm
Changed lines of the file:
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@@
 	(net 29 "Net-(R24-Pad2)")
 	(net 30 "unconnected-(U5-GPIO11{slash}TOUCH11{slash}ADC2_CH0{slash}FSPID{slash}FSPIIO5-Pad19)")
-	(net 31 "unconnected-(U5-GPIO8{slash}TOUCH8{slash}ADC1_CH7-Pad12)")
+	(net 31 "unconnected-(U5-GPIO46-Pad16)")
 	(net 32 "unconnected-(U5-GPIO17{slash}U1TXD{slash}ADC2_CH6{slash}DAC_1-Pad10)")
 	(net 33 "/I1_amp_a")
@@
 			)
 		)
-		(property "Value" "10k"
+		(property "Value" "dnp"
 			(at 0 -1.43 0)
 			(layer "B.Fab")
@@
 			)
 		)
-		(property "Value" "10k (1%)"
+		(property "Value" "4.7k (1%)"
 			(at 0 -1.43 0)
 			(layer "B.Fab")
@@
 			)
 		)
-		(property "Value" "100k (1%)"
+		(property "Value" "20k (1%)"
 			(at 0 -1.43 0)
 			(layer "B.Fab")
@@
 			)
 		)
-		(property "Value" "0.001"
+		(property "Value" "0.010"
 			(at 0 -2.62 90)
 			(layer "B.Fab")
@@
 			)
 		)
-		(property "Value" "20k"
+		(property "Value" "0"
 			(at 0 -1.43 0)
 			(layer "B.Fab")
@@
 			)
 		)
-		(property "Value" "10k"
+		(property "Value" "470"
 			(at 0 -1.43 0)
 			(layer "B.Fab")
@@
 			(size 1.5 0.9)
 			(layers "B.Cu" "B.Mask" "B.Paste")
-			(net 31 "unconnected-(U5-GPIO8{slash}TOUCH8{slash}ADC1_CH7-Pad12)")
+			(net 107 "PWR_C_SET_EN")
 			(pinfunction "GPIO8/TOUCH8/ADC1_CH7")
-			(pintype "bidirectional+no_connect")
+			(pintype "bidirectional")
 		)
 		(pad "13" smd rect
@@
 			(size 1.5 0.9)
 			(layers "B.Cu" "B.Mask" "B.Paste")
-			(net 107 "PWR_C_SET_EN")
+			(net 31 "unconnected-(U5-GPIO46-Pad16)")
 			(pinfunction "GPIO46")
-			(pintype "input")
+			(pintype "input+no_connect")
 		)
 		(pad "17" smd rect
@@
 			)
 		)
-		(property "Value" "0"
+		(property "Value" "100k (1%)"
 			(at 0 -1.43 0)
 			(layer "B.Fab")
@@
 			)
 		)
-		(property "Value" "10k"
+		(property "Value" "470"
 			(at 0 -1.43 90)
 			(layer "B.Fab")
@@
 			)
 		)
-		(property "Value" "22"
+		(property "Value" "dnp"
 			(at 0 -1.43 90)
 			(layer "B.Fab")
@@
 			)
 		)
-		(property "Value" "0.001"
+		(property "Value" "0.010"
 			(at 0 -2.62 90)
 			(layer "B.Fab")
@@
 			)
 		)
-		(property "Value" "0"
+		(property "Value" "10"
 			(at 0 -1.43 90)
 			(layer "B.Fab")
@@
 			)
 		)
-		(property "Value" "22"
+		(property "Value" "dnp"
 			(at 0 -1.43 90)
 			(layer "B.Fab")
@@
 	)
 	(segment
-		(start 127.1 77.58)
-		(end 126.61 78.07)
+		(start 121.63 75.54)
+		(end 121.63 76.8)
 		(width 0.2)
 		(layer "B.Cu")
@@
 	)
 	(segment
-		(start 126.61 79.22)
-		(end 125.995 79.835)
+		(start 122.48 74.69)
+		(end 121.63 75.54)
 		(width 0.2)
 		(layer "B.Cu")
@@
 	)
 	(segment
-		(start 132.16 79.58)
-		(end 130.16 77.58)
+		(start 135.28 97.69)
+		(end 132.872 95.282)
 		(width 0.2)
 		(layer "B.Cu")
@@
 	)
 	(segment
-		(start 171.62 97.69)
-		(end 135.28 97.69)
+		(start 132.872 84.422)
+		(end 132.16 83.71)
 		(width 0.2)
 		(layer "B.Cu")
@@
 	)
 	(segment
-		(start 132.872 95.282)
-		(end 132.872 84.422)
+		(start 177.29 95.8825)
+		(end 177.29 97.27)
 		(width 0.2)
 		(layer "B.Cu")
@@
 	)
 	(segment
-		(start 126.61 78.07)
-		(end 126.61 79.22)
+		(start 125.56 74.69)
+		(end 122.48 74.69)
 		(width 0.2)
 		(layer "B.Cu")
@@
 	)
 	(segment
-		(start 132.16 83.71)
-		(end 132.16 79.58)
+		(start 176.47 98.09)
+		(end 172.02 98.09)
 		(width 0.2)
 		(layer "B.Cu")
@@
 	)
 	(segment
-		(start 132.872 84.422)
-		(end 132.16 83.71)
+		(start 132.16 79.58)
+		(end 129.66 77.08)
 		(width 0.2)
 		(layer "B.Cu")
@@
 	)
 	(segment
-		(start 125.995 79.835)
-		(end 125.42 79.835)
+		(start 177.29 97.27)
+		(end 176.47 98.09)
 		(width 0.2)
 		(layer "B.Cu")
@@
 	)
 	(segment
-		(start 130.16 77.58)
-		(end 127.1 77.58)
+		(start 171.62 97.69)
+		(end 135.28 97.69)
 		(width 0.2)
 		(layer "B.Cu")
@@
 	)
 	(segment
-		(start 176.47 98.09)
-		(end 172.02 98.09)
+		(start 172.02 98.09)
+		(end 171.62 97.69)
 		(width 0.2)
 		(layer "B.Cu")
@@
 	)
 	(segment
-		(start 135.28 97.69)
-		(end 132.872 95.282)
+		(start 127.95 77.08)
+		(end 125.56 74.69)
 		(width 0.2)
 		(layer "B.Cu")
@@
 	)
 	(segment
-		(start 172.02 98.09)
-		(end 171.62 97.69)
+		(start 129.66 77.08)
+		(end 127.95 77.08)
 		(width 0.2)
 		(layer "B.Cu")
@@
 	)
 	(segment
-		(start 177.29 95.8825)
-		(end 177.29 97.27)
+		(start 132.872 95.282)
+		(end 132.872 84.422)
 		(width 0.2)
 		(layer "B.Cu")
@@
 	)
 	(segment
-		(start 177.29 97.27)
-		(end 176.47 98.09)
+		(start 132.16 83.71)
+		(end 132.16 79.58)
 		(width 0.2)
 		(layer "B.Cu")
