File: KiCad/ElectronicLoad.kicad_sch (KiCad schematic)
At the start: 162 parts, among them J1 LOAD, J4 12V, J5 USB, J6 PROG, M1 FAN, Q1 any, Q2 any, Q3 BSS138, Q4 PMOS, Q5 BSS138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

Commit message: rev 0.2 adjustments
Parts:
- R41: value 0 -> 100k (1%)
- R46: value 100k (1%) -> 20k (1%)
- R47: value 10k (1%) -> 4.7k (1%)
- R74: value 20k -> 0
- R75: value 10k -> dnp
- R81: value 0 -> 10
- R83, R84: value 10k -> 470
- RS1, RS2: value 0.001 -> 0.010
Other:
- note added: "*0-3.3V (12V)"
- note added: "*10k/20k for 12V supply"
- note added: "*5-100 mOhm"
- note added: "*TVS diodes to clamp voltages to 3.3V"
- note added: "*div by ~26.5"
- note added: "*div by ~5"
- note added: "*increase it in case of oscillations"
- note added: "~3.3 MHz bandwidth"
- note removed: "*div by 1"
- note removed: "*div by 48"
- note removed: "*or 10 / 100 mOhm"
Changed lines of the file:
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@@
 		)
 	)
-	(text "*or 10 / 100 mOhm"
+	(text "*5-100 mOhm"
 		(exclude_from_sim no)
 		(at 122.428 71.882 0)
@@
 	(text "*sets bandwidth with R9"
 		(exclude_from_sim no)
-		(at 91.694 56.388 0)
+		(at 84.836 52.832 0)
 		(effects
 			(font
-				(size 1.27 1.27)
+				(size 1.016 1.016)
 			)
 		)
 	)
-	(text "*0-10V"
+	(text "*0-3.3V (12V)"
 		(exclude_from_sim no)
-		(at 38.862 34.29 0)
+		(at 41.148 34.036 0)
 		(effects
 			(font
@@
 		)
 	)
+	(text "~3.3 MHz bandwidth"
+		(exclude_from_sim no)
+		(at 253.492 224.79 0)
+		(effects
+			(font
+				(size 1.016 1.016)
+			)
+		)
+	)
 	(text "*0-3V"
 		(exclude_from_sim no)
@@
 		)
 	)
-	(text "*div by 48"
+	(text "*TVS diodes to clamp\nvoltages to 3.3V"
 		(exclude_from_sim no)
-		(at 22.606 133.858 0)
+		(at 56.642 149.352 0)
 		(effects
 			(font
-				(size 1.27 1.27)
+				(size 1.016 1.016)
+			)
+			(justify right)
+		)
+	)
+	(text "*div by ~26.5"
+		(exclude_from_sim no)
+		(at 23.114 136.144 0)
+		(effects
+			(font
+				(size 1.016 1.016)
 			)
 		)
@@
 		)
 	)
+	(text "*increase it in case\n of oscillations"
+		(exclude_from_sim no)
+		(at 106.68 29.21 0)
+		(effects
+			(font
+				(size 1.016 1.016)
+			)
+			(justify right)
+		)
+	)
 	(text "1k (1%)"
 		(exclude_from_sim no)
@@
 		)
 	)
+	(text "*10k/20k for 12V supply"
+		(exclude_from_sim no)
+		(at 229.87 227.584 0)
+		(effects
+			(font
+				(size 1.016 1.016)
+			)
+		)
+	)
 	(text "Current Sense MCU"
 		(exclude_from_sim no)
@@
 		)
 	)
-	(text "*0-10V"
+	(text "*0-3.3V\n(12V)"
 		(exclude_from_sim no)
-		(at 49.276 65.278 0)
+		(at 52.578 65.532 0)
 		(effects
 			(font
 				(size 1.27 1.27)
 			)
+			(justify right)
 		)
 	)
-	(text "*div by 1"
+	(text "*div by ~5"
 		(exclude_from_sim no)
-		(at 22.352 122.428 0)
+		(at 24.13 123.444 0)
 		(effects
 			(font
-				(size 1.27 1.27)
+				(size 1.016 1.016)
 			)
 		)
@@
 			)
 		)
-		(property "Value" "10k (1%)"
+		(property "Value" "4.7k (1%)"
 			(at 23.368 143.764 0)
 			(effects
@@
 			)
 		)
-		(property "Value" "20k"
+		(property "Value" "0"
 			(at 232.918 225.044 90)
 			(effects
@@
 			)
 		)
-		(property "Value" "0"
-			(at 25.654 119.38 0)
+		(property "Value" "100k (1%)"
+			(at 23.114 119.634 0)
 			(effects
 				(font
@@
 			)
 		)
-		(property "Value" "10k"
+		(property "Value" "470"
 			(at 104.902 44.704 0)
 			(effects
@@
 		(dnp no)
 		(property "Reference" "C1"
-			(at 85.09 50.546 90)
+			(at 79.248 46.736 90)
 			(effects
 				(font
@@
 		)
 		(property "Value" "4.7nF"
-			(at 85.598 52.832 90)
+			(at 78.486 49.784 90)
 			(effects
 				(font
@@
 			)
 		)
-		(property "Value" "0"
+		(property "Value" "10"
 			(at 246.38 207.01 90)
 			(effects
@@
 			)
 		)
-		(property "Value" "0.001"
+		(property "Value" "0.010"
 			(at 126.238 68.834 0)
 			(effects
@@
 			)
 		)
-		(property "Value" "10k"
+		(property "Value" "dnp"
 			(at 215.392 227.33 0)
 			(effects
@@
 			)
 		)
-		(property "Value" "0.001"
+		(property "Value" "0.010"
 			(at 113.03 68.5799 0)
 			(effects
@@
 		(on_board yes)
 		(dnp no)
-		(fields_autoplaced yes)
 		(property "Reference" "R65"
 			(at 97.79 33.02 90)
@@
 			)
 		)
-		(property "Value" "100k (1%)"
+		(property "Value" "20k (1%)"
 			(at 22.86 129.54 0)
 			(effects
@@
 			)
 		)
-		(property "Value" "10k"
+		(property "Value" "470"
 			(at 138.938 44.704 0)
 			(effects

Commit message: rev 0.2 schematics + pcb adjustments
Parts:
- R52, R53: value 22 -> dnp
Connections:
- net PWR_C_SET_EN: now also U5.12 (GPIO8/TOUCH8/ADC1_CH7); no longer U5.16 (GPIO46)
Other:
- note added: "*div by X (for 12V supply)"
- note removed: "*div by X"
Changed lines of the file:
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@@
 		)
 	)
-	(text "*div by X"
+	(text "*div by X (for 12V supply)"
 		(exclude_from_sim no)
 		(at 200.914 121.412 0)
@@
 	)
 	(no_connect
-		(at 146.05 229.87)
+		(at 54.61 224.79)
 	)
 	(no_connect
@@
 	(wire
 		(pts
+			(xy 148.59 229.87) (xy 146.05 229.87)
+		)
+		(stroke
+			(width 0)
+			(type default)
+		)
+	)
+	(wire
+		(pts
 			(xy 240.03 45.72) (xy 240.03 50.8)
 		)
@@
 	(global_label "PWR_C_SET_EN"
 		(shape input)
-		(at 54.61 224.79 180)
+		(at 148.59 229.87 0)
 		(fields_autoplaced yes)
 		(effects
@@
 				(size 1.27 1.27)
 			)
-			(justify right)
+			(justify left)
 		)
 		(property "Intersheetrefs" "${INTERSHEET_REFS}"
-			(at 37.655 224.79 0)
+			(at 165.545 229.87 0)
 			(effects
 				(font
 					(size 1.27 1.27)
 				)
-				(justify right)
+				(justify left)
 				(hide yes)
 			)
@@
 			)
 		)
-		(property "Value" "22"
+		(property "Value" "dnp"
 			(at 202.946 130.556 0)
 			(effects
@@
 			)
 		)
-		(property "Value" "22"
+		(property "Value" "dnp"
 			(at 202.946 143.256 0)
 			(effects
